File: eagle/doppler-tiny.brd (EAGLE design)
At the start: 67 x 27 mm, 46 parts, among them U1 Tiny45-20-SMT, U2 AUREL-TX-FM-MID, U3 ADP160, U4 MAG3110FCR1, U5 SS39ET, X2 PYRO

Commit message: Add files via upload
Parts:
- added JP13, JP14: STRAP, pinhead:1X01
- added SJ1: (no value), SparkFun-Passives:PAD-JUMPER-2-NO_NO_SILK
- moved JP12 29.5 mm to (27.9, 5.71)
- moved JP8 10.0 mm to (37.5, 5.08)
- moved JP2 0.64 mm to (37.5, 7.62)
- moved JP1 0.63 mm to (42.5, 7.62)
- moved JP6 0.16 mm to (33.0, 5.71)
Connections:
- new net N$9: G1.-, SJ1.1
- net GND: now also JP13.1, JP14.1
- net N$3: now also SJ1.2; no longer G1.-
Routing:
- net N$3: track 8.05 -> 5.29 mm
- net VBAT: track 119.7 -> 120.4 mm
- added copper zone on layer 1, net N$7
Other:
- board text added: "Pyro Doppler"
Changed lines of the file:
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@@
 <layer number="23" name="tOrigins" color="15" fill="1" visible="yes" active="yes"/>
 <layer number="24" name="bOrigins" color="15" fill="1" visible="yes" active="yes"/>
-<layer number="25" name="tNames" color="7" fill="1" visible="yes" active="yes"/>
-<layer number="26" name="bNames" color="7" fill="1" visible="yes" active="yes"/>
+<layer number="25" name="tNames" color="7" fill="1" visible="no" active="yes"/>
+<layer number="26" name="bNames" color="7" fill="1" visible="no" active="yes"/>
 <layer number="27" name="tValues" color="7" fill="1" visible="no" active="yes"/>
 <layer number="28" name="bValues" color="7" fill="1" visible="no" active="yes"/>
@@
 <circle x="64" y="24" radius="3.1" width="0.4064" layer="41"/>
 <circle x="50" y="3" radius="3.1" width="0.4064" layer="41"/>
+<text x="52.705" y="21.59" size="1.778" layer="41" font="vector" ratio="18" rot="SR180" align="center">Pyro
+Doppler</text>
 </plain>
 <attributes>
@@
 <element name="C2" library="rcl" package="C0603" value="100n" x="65.405" y="3.175" rot="R270"/>
 <element name="G1" library="rotary-launcher" package="CRAA" value="CR-AA" x="49.53" y="13.335" rot="MR180"/>
-<element name="JP1" library="pinhead" package="1X01" value="ENA+" x="43.18" y="7.62" rot="R270"/>
-<element name="JP6" library="pinhead" package="1X01" value="GR_LED" x="33.02" y="5.87375"/>
+<element name="JP1" library="pinhead" package="1X01" value="ENA+" x="42.545" y="7.62" rot="R270"/>
+<element name="JP6" library="pinhead" package="1X01" value="GR_LED" x="33.02" y="5.715"/>
 <element name="JP10" library="pinhead" package="1X01" value="GND" x="13.335" y="3.175"/>
 <element name="JP9" library="pinhead" package="1X01" value="ARM+" x="10.795" y="3.175"/>
-<element name="JP2" library="pinhead" package="1X01" value="ENA-" x="36.83" y="7.62" rot="R270"/>
+<element name="JP2" library="pinhead" package="1X01" value="ENA-" x="37.465" y="7.62" rot="R270"/>
 <element name="JP3" library="pinhead" package="1X01" value="!RES" x="18.0975" y="17.145"/>
 <element name="JP4" library="pinhead" package="1X01" value="MOSI" x="30.48" y="8.73125"/>
 <element name="JP5" library="pinhead" package="1X01" value="MISO" x="30.48" y="11.27125"/>
 <element name="JP7" library="pinhead" package="1X01" value="SCK" x="32.385" y="13.81125"/>
-<element name="JP8" library="pinhead" package="1X01" value="GND" x="27.46375" y="5.715"/>
+<element name="JP8" library="pinhead" package="1X01" value="GND" x="37.465" y="5.08"/>
 <element name="LED1" library="led" package="CHIPLED_0805" value="" x="30.32125" y="5.715" rot="R90"/>
 <element name="Q2" library="SparkFun-DiscreteSemi" package="SOT23-3" value="" x="9.525" y="7.62" rot="R90">
@@
 <element name="R10" library="rcl" package="R0603" value="10k" x="29.845" y="14.44625" rot="R270"/>
 <element name="JP11" library="pinhead" package="1X01" value="SDA_VIA" x="32.54375" y="16.51" rot="R270"/>
-<element name="JP12" library="pinhead" package="1X01" value="GND" x="31.75" y="34.925" rot="R180"/>
+<element name="JP12" library="pinhead" package="1X01" value="GND" x="27.94" y="5.715" rot="R180"/>
 <element name="R11" library="rcl" package="R1206" value="" x="40.005" y="22.86" rot="R180"/>
+<element name="JP13" library="pinhead" package="1X01" value="STRAP" x="45.085" y="22.225"/>
+<element name="JP14" library="pinhead" package="1X01" value="STRAP" x="45.085" y="3.81"/>
+<element name="SJ1" library="SparkFun-Passives" package="PAD-JUMPER-2-NO_NO_SILK" value="" x="36.83" y="10.795" rot="R270"/>
 </elements>
 <signals>
@@
 <contactref element="X1" pad="GND@4"/>
 <contactref element="C6" pad="-"/>
-<polygon width="0.4064" layer="1" isolate="0.4064" orphans="yes">
+<polygon width="0.4064" layer="1" isolate="0.4064">
 <vertex x="-0.635" y="-0.635"/>
 <vertex x="67.945" y="-0.635"/>
@@
 <wire x1="38.583" y1="22.86" x2="36.9325" y2="22.86" width="0.4064" layer="1"/>
 <wire x1="36.9325" y1="22.86" x2="36.5125" y2="22.44" width="0.4064" layer="1"/>
-<wire x1="31.37625" y1="22.70125" x2="31.75" y2="34.925" width="0" layer="19" extent="1-1"/>
-<wire x1="41.427" y1="22.86" x2="38.583" y2="22.86" width="0" layer="19" extent="1-1"/>
+<contactref element="JP13" pad="1"/>
+<contactref element="JP14" pad="1"/>
 <wire x1="60.96" y1="2.032" x2="60.96" y2="2.032" width="0" layer="19" extent="1-16"/>
 <wire x1="55.88" y1="2.032" x2="55.88" y2="3.81" width="0" layer="19" extent="16-16"/>
+<wire x1="38.583" y1="22.86" x2="41.427" y2="22.86" width="0" layer="19" extent="1-1"/>
 </signal>
 <signal name="SCL">
@@
 <contactref element="LED1" pad="A"/>
 <contactref element="JP6" pad="1"/>
-<wire x1="33.02" y1="9.6275" x2="33.02" y2="5.87375" width="0.4064" layer="1"/>
-<wire x1="31.37125" y1="5.715" x2="32.86125" y2="5.715" width="0.4064" layer="1"/>
-<wire x1="32.86125" y1="5.715" x2="33.02" y2="5.87375" width="0.4064" layer="1"/>
+<wire x1="33.02" y1="9.6275" x2="33.02" y2="5.715" width="0.4064" layer="1"/>
+<wire x1="31.37125" y1="5.715" x2="33.02" y2="5.715" width="0.4064" layer="1"/>
 </signal>
 <signal name="N$138">
 <contactref element="Q2" pad="3"/>
 <contactref element="X2" pad="1"/>
-<wire x1="8.425" y1="7.62" x2="6.985" y2="7.62" width="0.4064" layer="1"/>
-<wire x1="6.985" y1="7.62" x2="5.08" y2="9.525" width="0.4064" layer="1"/>
-<wire x1="5.08" y1="9.525" x2="5.08" y2="11.43" width="0.4064" layer="1"/>
+<wire x1="8.425" y1="7.62" x2="6.985" y2="7.62" width="1.27" layer="1"/>
+<wire x1="6.985" y1="7.62" x2="5.08" y2="9.525" width="1.27" layer="1"/>
+<wire x1="5.08" y1="9.525" x2="5.08" y2="11.43" width="1.27" layer="1"/>
 </signal>
 <signal name="GR_LED">
@@
 <wire x1="45.085" y1="6.35" x2="45.085" y2="10.21625" width="0.4064" layer="1"/>
 <wire x1="45.085" y1="10.21625" x2="44.82375" y2="10.4775" width="0.4064" layer="1"/>
-<wire x1="44.82375" y1="10.4775" x2="44.82375" y2="19.31125" width="0.4064" layer="1"/>
-<wire x1="44.82375" y1="19.31125" x2="43.18" y2="20.955" width="0.4064" layer="1"/>
-<wire x1="43.18" y1="20.955" x2="40.005" y2="20.955" width="0.4064" layer="1"/>
-<wire x1="40.005" y1="20.955" x2="36.7275" y2="20.955" width="0.4064" layer="1"/>
+<wire x1="40.005" y1="20.955" x2="39.37" y2="20.955" width="0.4064" layer="1"/>
+<wire x1="39.37" y1="20.955" x2="36.7275" y2="20.955" width="0.4064" layer="1"/>
 <wire x1="36.7275" y1="20.955" x2="36.5125" y2="20.74" width="0.4064" layer="1"/>
 <wire x1="26.9875" y1="21.9075" x2="29.845" y2="24.765" width="0.4064" layer="1"/>
@@
 <wire x1="26.6675" y1="20.30875" x2="26.6675" y2="21.905" width="0.4064" layer="1"/>
 <wire x1="26.6675" y1="21.905" x2="26.67" y2="21.9075" width="0.4064" layer="1"/>
+<wire x1="44.82375" y1="10.4775" x2="44.82375" y2="11.69125" width="0.4064" layer="1"/>
+<wire x1="44.82375" y1="11.69125" x2="43.815" y2="12.7" width="0.4064" layer="1"/>
+<wire x1="43.815" y1="12.7" x2="40.005" y2="12.7" width="0.4064" layer="1"/>
+<wire x1="40.005" y1="12.7" x2="39.37" y2="13.335" width="0.4064" layer="1"/>
+<wire x1="39.37" y1="13.335" x2="39.37" y2="20.955" width="0.4064" layer="1"/>
 </signal>
 <signal name="N$2">
@@
 <wire x1="40.955" y1="10.525" x2="43.07625" y2="10.525" width="0.4064" layer="1"/>
 <wire x1="43.07625" y1="10.525" x2="43.12375" y2="10.4775" width="0.4064" layer="1"/>
-<wire x1="43.12375" y1="10.4775" x2="43.12375" y2="7.67625" width="0.4064" layer="1"/>
-<wire x1="43.12375" y1="7.67625" x2="43.18" y2="7.62" width="0.4064" layer="1"/>
+<wire x1="43.12375" y1="10.4775" x2="43.12375" y2="8.19875" width="0.4064" layer="1"/>
+<wire x1="43.12375" y1="8.19875" x2="42.545" y2="7.62" width="0.4064" layer="1"/>
 </signal>
 <signal name="N$3">
 <contactref element="JP2" pad="1"/>
 <contactref element="Q1" pad="2"/>
-<contactref element="G1" pad="-"/>
-<wire x1="36.83" y1="13.335" x2="36.83" y2="10.795" width="0.4064" layer="1"/>
-<wire x1="36.83" y1="10.795" x2="36.83" y2="7.62" width="0.4064" layer="1"/>
-<wire x1="39.055" y1="10.525" x2="37.1" y2="10.525" width="0.4064" layer="1"/>
-<wire x1="37.1" y1="10.525" x2="36.83" y2="10.795" width="0.4064" layer="1"/>
+<contactref element="SJ1" pad="2"/>
+<wire x1="36.83" y1="10.345" x2="38.875" y2="10.345" width="0.4064" layer="1"/>
+<wire x1="38.875" y1="10.345" x2="39.055" y2="10.525" width="0.4064" layer="1"/>
+<wire x1="37.465" y1="7.62" x2="37.465" y2="9.71" width="0.4064" layer="1"/>
+<wire x1="37.465" y1="9.71" x2="36.83" y2="10.345" width="0.4064" layer="1"/>
 </signal>
 <signal name="VPYRO">
@@
 <contactref element="C6" pad="+"/>
 <contactref element="X2" pad="2"/>
-<wire x1="12.065" y1="15.748" x2="5.842" y2="15.748" width="0.4064" layer="1"/>
-<wire x1="5.842" y1="15.748" x2="5.08" y2="16.51" width="0.4064" layer="1"/>
+<wire x1="12.065" y1="15.748" x2="5.842" y2="15.748" width="1.27" layer="1"/>
+<wire x1="5.842" y1="15.748" x2="5.08" y2="16.51" width="1.27" layer="1"/>
 <wire x1="12.1" y1="17.565" x2="12.1" y2="15.783" width="0.4064" layer="1"/>
 <wire x1="12.1" y1="15.783" x2="12.065" y2="15.748" width="0.4064" layer="1"/>
@@
 <wire x1="23.1775" y1="19.84375" x2="23.1775" y2="18.3125" width="0.4064" layer="1"/>
 </signal>
+<signal name="N$7">
+<polygon width="0.01" layer="1">
+<vertex x="46.355" y="25.4"/>
+<vertex x="59.69" y="25.4"/>
+<vertex x="59.69" y="18.415"/>
+<vertex x="46.355" y="18.415"/>
+</polygon>
+</signal>
+<signal name="N$9">
+<contactref element="G1" pad="-"/>
+<contactref element="SJ1" pad="1"/>
+<wire x1="36.83" y1="11.245" x2="36.83" y2="13.335" width="0" layer="19" extent="1-1"/>
+</signal>
 </signals>
 </board>
 </drawing>
+<compatibility>
+<note version="6.3" minversion="6.2.2" severity="warning">
+Since Version 6.2.2 text objects can contain more than one line,
+which will not be processed correctly with this version.
+</note>
+</compatibility>
 </eagle>

Commit message: Add files via upload
Parts:
- added JP15, JP16: STRAP, pinhead:1X01
- moved C7 4.26 mm to (10.8, 11.4)
- moved Q2 4.02 mm to (8.26, 11.4)
- moved R7 3.86 mm to (14.0, 11.4)
- moved JP10 3.81 mm to (13.3, 6.99)
- moved JP9 3.81 mm to (10.8, 6.99)
- moved JP3 0.63 mm to (18.1, 16.5)
Connections:
- net GND: now also JP15.1, JP16.1
Routing:
- net N$138: track 6.04 -> 2.08 mm
- net GND: track 5.07 -> 8.94 mm
- net N$133: track 14.2 -> 10.9 mm
- net PYRO: track 2.76 -> 4.85 mm
- net N$5: track 0.00 -> 1.78 mm
Changed lines of the file:
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@@
 </autorouter>
 <elements>
-<element name="C7" library="rcl" package="C0603" value="100n" x="12.7" y="7.62" rot="R90"/>
+<element name="C7" library="rcl" package="C0603" value="100n" x="10.795" y="11.43" rot="R90"/>
 <element name="C5" library="rcl" package="C0603" value="1uF" x="12.065" y="21.74875" rot="R90"/>
 <element name="C1" library="rcl" package="C0603" value="100n" x="22.225" y="8.73125" rot="R180"/>
@@
 <element name="JP1" library="pinhead" package="1X01" value="ENA+" x="42.545" y="7.62" rot="R270"/>
 <element name="JP6" library="pinhead" package="1X01" value="GR_LED" x="33.02" y="5.715"/>
-<element name="JP10" library="pinhead" package="1X01" value="GND" x="13.335" y="3.175"/>
-<element name="JP9" library="pinhead" package="1X01" value="ARM+" x="10.795" y="3.175"/>
+<element name="JP10" library="pinhead" package="1X01" value="GND" x="13.335" y="6.985"/>
+<element name="JP9" library="pinhead" package="1X01" value="ARM+" x="10.795" y="6.985"/>
 <element name="JP2" library="pinhead" package="1X01" value="ENA-" x="37.465" y="7.62" rot="R270"/>
-<element name="JP3" library="pinhead" package="1X01" value="!RES" x="18.0975" y="17.145"/>
+<element name="JP3" library="pinhead" package="1X01" value="!RES" x="18.0975" y="16.51"/>
 <element name="JP4" library="pinhead" package="1X01" value="MOSI" x="30.48" y="8.73125"/>
 <element name="JP5" library="pinhead" package="1X01" value="MISO" x="30.48" y="11.27125"/>
@@
 <element name="JP8" library="pinhead" package="1X01" value="GND" x="37.465" y="5.08"/>
 <element name="LED1" library="led" package="CHIPLED_0805" value="" x="30.32125" y="5.715" rot="R90"/>
-<element name="Q2" library="SparkFun-DiscreteSemi" package="SOT23-3" value="" x="9.525" y="7.62" rot="R90">
-<attribute name="PROD_ID" value="TRANS-08345" x="9.525" y="7.62" size="1.778" layer="27" rot="R90" display="off"/>
+<element name="Q2" library="SparkFun-DiscreteSemi" package="SOT23-3" value="" x="8.255" y="11.43" rot="R90">
+<attribute name="PROD_ID" value="TRANS-08345" x="8.255" y="11.43" size="1.778" layer="27" rot="R90" display="off"/>
 </element>
 <element name="Q1" library="SparkFun-DiscreteSemi" package="SOT23-3" value="" x="40.005" y="9.525" rot="R180">
@@
 </element>
 <element name="R1" library="rcl" package="R0603" value="100k" x="43.97375" y="10.4775"/>
-<element name="R7" library="rcl" package="R0603" value="6k8" x="14.605" y="7.62" rot="R270"/>
+<element name="R7" library="rcl" package="R0603" value="6k8" x="13.97" y="11.43" rot="R270"/>
 <element name="R2" library="rcl" package="R0603" value="10k" x="20.47875" y="17.93875" rot="R270"/>
 <element name="R4" library="rcl" package="R0603" value="470" x="12.1" y="18.415" rot="R270"/>
@@
 <element name="JP14" library="pinhead" package="1X01" value="STRAP" x="45.085" y="3.81"/>
 <element name="SJ1" library="SparkFun-Passives" package="PAD-JUMPER-2-NO_NO_SILK" value="" x="36.83" y="10.795" rot="R270"/>
+<element name="JP15" library="pinhead" package="1X01" value="STRAP" x="18.415" y="19.05"/>
+<element name="JP16" library="pinhead" package="1X01" value="STRAP" x="18.415" y="8.89"/>
 </elements>
 <signals>
@@
 <contactref element="JP13" pad="1"/>
 <contactref element="JP14" pad="1"/>
+<wire x1="16.5401" y1="21.74875" x2="17.30375" y2="21.74875" width="0.4064" layer="1"/>
+<wire x1="17.30375" y1="21.74875" x2="18.415" y2="22.86" width="0.4064" layer="1"/>
+<wire x1="31.75" y1="17.78" x2="31.115" y2="17.78" width="0.4064" layer="1"/>
+<wire x1="31.115" y1="17.78" x2="30.48" y2="17.145" width="0.4064" layer="1"/>
+<contactref element="JP15" pad="1"/>
+<contactref element="JP16" pad="1"/>
 <wire x1="60.96" y1="2.032" x2="60.96" y2="2.032" width="0" layer="19" extent="1-16"/>
 <wire x1="55.88" y1="2.032" x2="55.88" y2="3.81" width="0" layer="19" extent="16-16"/>
@@
 <wire x1="18.0975" y1="15.1375" x2="20.06055" y2="15.1375" width="0.4064" layer="1"/>
 <wire x1="20.06055" y1="15.1375" x2="20.7518" y2="14.44625" width="0.4064" layer="1"/>
-<wire x1="18.0975" y1="15.1375" x2="18.0975" y2="17.145" width="0.4064" layer="1"/>
+<wire x1="18.0975" y1="15.1375" x2="18.0975" y2="16.51" width="0.4064" layer="1"/>
 <wire x1="15.71625" y1="17.0425" x2="17.995" y2="17.0425" width="0.4064" layer="1"/>
-<wire x1="17.995" y1="17.0425" x2="18.0975" y2="17.145" width="0.4064" layer="1"/>
+<wire x1="17.995" y1="17.0425" x2="18.0975" y2="16.51" width="0.4064" layer="1"/>
 <wire x1="20.47875" y1="17.08875" x2="20.47875" y2="15.5557" width="0.4064" layer="1"/>
 <wire x1="20.47875" y1="15.5557" x2="20.06055" y2="15.1375" width="0.4064" layer="1"/>
@@
 <wire x1="20.7518" y1="13.17625" x2="18.35875" y2="13.17625" width="0.4064" layer="1"/>
 <wire x1="18.35875" y1="13.17625" x2="18.0975" y2="13.4375" width="0.4064" layer="1"/>
-<wire x1="16.03375" y1="13.39125" x2="18.0975" y2="13.4375" width="0" layer="19" extent="1-1"/>
+<wire x1="16.03375" y1="13.39125" x2="18.05125" y2="13.39125" width="0.4064" layer="1"/>
+<wire x1="18.05125" y1="13.39125" x2="18.0975" y2="13.4375" width="0.4064" layer="1"/>
 </signal>
 <signal name="N$133">
@@
 <contactref element="JP9" pad="1"/>
 <contactref element="C7" pad="1"/>
-<wire x1="14.605" y1="6.77" x2="12.7" y2="6.77" width="0.4064" layer="1"/>
-<wire x1="12.7" y1="6.77" x2="10.625" y2="6.77" width="0.4064" layer="1"/>
-<wire x1="10.625" y1="6.77" x2="10.525" y2="6.67" width="0.4064" layer="1"/>
-<wire x1="10.795" y1="3.175" x2="10.795" y2="6.4" width="0.4064" layer="1"/>
-<wire x1="10.795" y1="6.4" x2="10.525" y2="6.67" width="0.4064" layer="1"/>
-<wire x1="14.605" y1="6.77" x2="15.81875" y2="6.77" width="0.4064" layer="1"/>
-<wire x1="15.81875" y1="6.77" x2="16.35125" y2="7.3025" width="0.4064" layer="1"/>
-<wire x1="16.35125" y1="7.3025" x2="16.35125" y2="11.37375" width="0.4064" layer="1"/>
-<wire x1="16.35125" y1="11.37375" x2="16.03375" y2="11.69125" width="0.4064" layer="1"/>
+<wire x1="13.97" y1="10.58" x2="14.9225" y2="10.58" width="0.4064" layer="1"/>
+<wire x1="14.9225" y1="10.58" x2="16.03375" y2="11.69125" width="0.4064" layer="1"/>
+<wire x1="13.97" y1="10.58" x2="10.795" y2="10.58" width="0.4064" layer="1"/>
+<wire x1="9.255" y1="10.48" x2="10.695" y2="10.48" width="0.4064" layer="1"/>
+<wire x1="10.695" y1="10.48" x2="10.795" y2="10.58" width="0.4064" layer="1"/>
+<wire x1="10.795" y1="10.58" x2="10.795" y2="6.985" width="0.4064" layer="1"/>
 </signal>
 <signal name="N$137">
@@
 <contactref element="Q2" pad="3"/>
 <contactref element="X2" pad="1"/>
-<wire x1="8.425" y1="7.62" x2="6.985" y2="7.62" width="1.27" layer="1"/>
-<wire x1="6.985" y1="7.62" x2="5.08" y2="9.525" width="1.27" layer="1"/>
-<wire x1="5.08" y1="9.525" x2="5.08" y2="11.43" width="1.27" layer="1"/>
+<wire x1="7.155" y1="11.43" x2="5.08" y2="11.43" width="1.27" layer="1"/>
 </signal>
 <signal name="GR_LED">
@@
 <contactref element="C6" pad="+"/>
 <contactref element="X2" pad="2"/>
-<wire x1="12.065" y1="15.748" x2="5.842" y2="15.748" width="1.27" layer="1"/>
-<wire x1="5.842" y1="15.748" x2="5.08" y2="16.51" width="1.27" layer="1"/>
 <wire x1="12.1" y1="17.565" x2="12.1" y2="15.783" width="0.4064" layer="1"/>
 <wire x1="12.1" y1="15.783" x2="12.065" y2="15.748" width="0.4064" layer="1"/>
+<wire x1="5.08" y1="16.51" x2="11.303" y2="16.51" width="1.27" layer="1"/>
+<wire x1="11.303" y1="16.51" x2="12.065" y2="15.748" width="1.27" layer="1"/>
 </signal>
 <signal name="N$1">
@@
 <contactref element="U2" pad="4"/>
 <contactref element="X1" pad="P"/>
-<wire x1="58.42" y1="2.032" x2="58.42" y2="3.81" width="0" layer="19" extent="1-1"/>
+<wire x1="58.42" y1="3.81" x2="58.42" y2="2.032" width="0.4064" layer="1"/>
 </signal>
 <signal name="SDA">
