File: eagle/doppler-tiny.sch (EAGLE design)
At the start: 46 parts, among them Q1 MOSFET-NCHANNELBSS123LT1G, Q2 MOSFET-NCHANNELBSS123LT1G, U1 Tiny45-20-SMT, U2 AUREL-TX-FM-MID, U3 ADP160, U4 MAG3110FCR1, U5 SS39ET, X2 PYRO

Commit message: Add files via upload
Parts:
- added JP13, JP14: STRAP, pinhead:PINHD-1X1
- added SJ1: JUMPER-PAD-2-NO, SparkFun-Passives:JUMPER-PAD-2-NO
Connections:
- new net N$9: G1.-, SJ1.1
- net GND: now also JP13.1, JP14.1
- net N$3: now also SJ1.2; no longer G1.-
Changed lines of the file:
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@@
 <part name="GND25" library="supply1" deviceset="GND" device=""/>
 <part name="GND26" library="supply1" deviceset="GND" device=""/>
+<part name="GND27" library="supply1" deviceset="GND" device=""/>
+<part name="JP13" library="pinhead" deviceset="PINHD-1X1" device="" value="STRAP"/>
+<part name="JP14" library="pinhead" deviceset="PINHD-1X1" device="" value="STRAP"/>
+<part name="SJ1" library="SparkFun-Passives" deviceset="JUMPER-PAD-2-NO" device="" value=""/>
 </parts>
 <sheets>
@@
 <instance part="GND25" gate="1" x="124.46" y="78.74"/>
 <instance part="GND26" gate="1" x="139.7" y="78.74"/>
+<instance part="GND27" gate="1" x="248.92" y="137.16"/>
+<instance part="JP13" gate="G$1" x="241.3" y="144.78" rot="R180"/>
+<instance part="JP14" gate="G$1" x="241.3" y="154.94" rot="R180"/>
+<instance part="SJ1" gate="G$1" x="25.4" y="134.62"/>
 </instances>
 <busses>
@@
 <wire x1="137.16" y1="83.82" x2="139.7" y2="83.82" width="0.1524" layer="91"/>
 <wire x1="139.7" y1="83.82" x2="139.7" y2="81.28" width="0.1524" layer="91"/>
+</segment>
+<segment>
+<pinref part="GND27" gate="1" pin="GND"/>
+<wire x1="243.84" y1="144.78" x2="248.92" y2="144.78" width="0.1524" layer="91"/>
+<wire x1="248.92" y1="144.78" x2="248.92" y2="139.7" width="0.1524" layer="91"/>
+<pinref part="JP13" gate="G$1" pin="1"/>
+<pinref part="JP14" gate="G$1" pin="1"/>
+<wire x1="243.84" y1="154.94" x2="248.92" y2="154.94" width="0.1524" layer="91"/>
+<wire x1="248.92" y1="154.94" x2="248.92" y2="144.78" width="0.1524" layer="91"/>
+<junction x="248.92" y="144.78"/>
 </segment>
 </net>
@@
 <wire x1="50.8" y1="139.7" x2="50.8" y2="134.62" width="0.1524" layer="91"/>
 <junction x="50.8" y="139.7"/>
-<pinref part="G1" gate="1" pin="-"/>
-<wire x1="50.8" y1="134.62" x2="15.24" y2="134.62" width="0.1524" layer="91"/>
-<wire x1="15.24" y1="134.62" x2="15.24" y2="149.86" width="0.1524" layer="91"/>
+<pinref part="SJ1" gate="G$1" pin="2"/>
+<wire x1="30.48" y1="134.62" x2="50.8" y2="134.62" width="0.1524" layer="91"/>
 </segment>
 </net>
@@
 </segment>
 </net>
+<net name="N$9" class="0">
+<segment>
+<pinref part="G1" gate="1" pin="-"/>
+<wire x1="15.24" y1="134.62" x2="15.24" y2="149.86" width="0.1524" layer="91"/>
+<pinref part="SJ1" gate="G$1" pin="1"/>
+<wire x1="20.32" y1="134.62" x2="15.24" y2="134.62" width="0.1524" layer="91"/>
+</segment>
+</net>

Commit message: Add files via upload
Parts:
- added JP15, JP16: STRAP, pinhead:PINHD-1X1
Connections:
- net GND: now also JP15.1, JP16.1
Changed lines of the file:
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@@
 <part name="JP14" library="pinhead" deviceset="PINHD-1X1" device="" value="STRAP"/>
 <part name="SJ1" library="SparkFun-Passives" deviceset="JUMPER-PAD-2-NO" device="" value=""/>
+<part name="GND28" library="supply1" deviceset="GND" device=""/>
+<part name="JP15" library="pinhead" deviceset="PINHD-1X1" device="" value="STRAP"/>
+<part name="JP16" library="pinhead" deviceset="PINHD-1X1" device="" value="STRAP"/>
 </parts>
 <sheets>
@@
 <instance part="JP14" gate="G$1" x="241.3" y="154.94" rot="R180"/>
 <instance part="SJ1" gate="G$1" x="25.4" y="134.62"/>
+<instance part="GND28" gate="1" x="236.22" y="137.16"/>
+<instance part="JP15" gate="G$1" x="228.6" y="144.78" rot="R180"/>
+<instance part="JP16" gate="G$1" x="228.6" y="154.94" rot="R180"/>
 </instances>
 <busses>
@@
 <junction x="248.92" y="144.78"/>
 </segment>
+<segment>
+<pinref part="GND28" gate="1" pin="GND"/>
+<wire x1="231.14" y1="144.78" x2="236.22" y2="144.78" width="0.1524" layer="91"/>
+<wire x1="236.22" y1="144.78" x2="236.22" y2="139.7" width="0.1524" layer="91"/>
+<pinref part="JP15" gate="G$1" pin="1"/>
+<pinref part="JP16" gate="G$1" pin="1"/>
+<wire x1="231.14" y1="154.94" x2="236.22" y2="154.94" width="0.1524" layer="91"/>
+<wire x1="236.22" y1="154.94" x2="236.22" y2="144.78" width="0.1524" layer="91"/>
+<junction x="236.22" y="144.78"/>
+</segment>
 </net>
